File: skateboard_main_controller_kicad/skateboard_main_controller_kicad.kicad_sch (KiCad schematic)
At the start: 18 parts, among them J1 Conn_01x02_Socket, J2 Conn_01x06_Socket, J3 Conn_01x01_Socket, J4 Conn_01x01_Socket, U1 STM32F103C8T6TR

Commit message: add correct kicad files
Other:
- note added: "4/1/2026"
- note added: "Juanpablo Mora"
- note added: "skateboard controller test board"
Changed lines of the file:
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@@
+    (effects (font (size 1.27 1.27)) (justify left bottom))
+  )
+  (text "4/1/2026" (at 503.555 403.86 0)
+    (effects (font (size 1.27 1.27)) (justify left bottom))
+  )
+  (text "skateboard controller test board" (at 483.87 400.05 0)
     (effects (font (size 1.27 1.27)) (justify left bottom))
   )
@@
   (text "vdd power block" (at 396.24 182.88 0)
     (effects (font (size 1.27 1.27)) (justify left bottom))
+  )
+  (text "Juanpablo Mora" (at 490.22 386.715 0)
+    (effects (font (size 6 6)) (justify left bottom))
   )
   (global_label "SPI_CS" (shape output) (at 227.965 189.865 180) (fields_autoplaced)
@@
     (pin "2")
     (instances
-      (project "skateboard_main_controller"
+      (project "skateboard_main_controller_kicad"
         (path "/729eee83-acb9-4794-a583-aef43df0c6ef"
           (reference "C5") (unit 1)
@@
     (pin "2")
     (instances
-      (project "skateboard_main_controller"
+      (project "skateboard_main_controller_kicad"
         (path "/729eee83-acb9-4794-a583-aef43df0c6ef"
           (reference "C6") (unit 1)
@@
     (pin "1")
     (instances
-      (project "skateboard_main_controller"
+      (project "skateboard_main_controller_kicad"
         (path "/729eee83-acb9-4794-a583-aef43df0c6ef"
           (reference "TP1") (unit 1)
@@
     (pin "1")
     (instances
-      (project "skateboard_main_controller"
+      (project "skateboard_main_controller_kicad"
         (path "/729eee83-acb9-4794-a583-aef43df0c6ef"
           (reference "TP4") (unit 1)
@@
     (pin "1")
     (instances
-      (project "skateboard_main_controller"
+      (project "skateboard_main_controller_kicad"
         (path "/729eee83-acb9-4794-a583-aef43df0c6ef"
           (reference "#PWR03") (unit 1)
@@
     (pin "1")
     (instances
-      (project "skateboard_main_controller"
+      (project "skateboard_main_controller_kicad"
         (path "/729eee83-acb9-4794-a583-aef43df0c6ef"
           (reference "#PWR010") (unit 1)
@@
     (pin "1")
     (instances
-      (project "skateboard_main_controller"
+      (project "skateboard_main_controller_kicad"
         (path "/729eee83-acb9-4794-a583-aef43df0c6ef"
           (reference "TP3") (unit 1)
@@
     (pin "1")
     (instances
-      (project "skateboard_main_controller"
+      (project "skateboard_main_controller_kicad"
         (path "/729eee83-acb9-4794-a583-aef43df0c6ef"
           (reference "J3") (unit 1)
@@
     (pin "2")
     (instances
-      (project "skateboard_main_controller"
+      (project "skateboard_main_controller_kicad"
         (path "/729eee83-acb9-4794-a583-aef43df0c6ef"
           (reference "J1") (unit 1)
@@
     (pin "2")
     (instances
-      (project "skateboard_main_controller"
+      (project "skateboard_main_controller_kicad"
         (path "/729eee83-acb9-4794-a583-aef43df0c6ef"
           (reference "C7") (unit 1)
@@
     (pin "1")
     (instances
-      (project "skateboard_main_controller"
+      (project "skateboard_main_controller_kicad"
         (path "/729eee83-acb9-4794-a583-aef43df0c6ef"
           (reference "#PWR05") (unit 1)
@@
     (pin "2")
     (instances
-      (project "skateboard_main_controller"
+      (project "skateboard_main_controller_kicad"
         (path "/729eee83-acb9-4794-a583-aef43df0c6ef"
           (reference "C4") (unit 1)
@@
     (pin "9")
     (instances
-      (project "skateboard_main_controller"
+      (project "skateboard_main_controller_kicad"
         (path "/729eee83-acb9-4794-a583-aef43df0c6ef"
           (reference "U1") (unit 1)
@@
     (pin "1")
     (instances
-      (project "skateboard_main_controller"
+      (project "skateboard_main_controller_kicad"
         (path "/729eee83-acb9-4794-a583-aef43df0c6ef"
           (reference "#PWR011") (unit 1)
@@
     (pin "2")
     (instances
-      (project "skateboard_main_controller"
+      (project "skateboard_main_controller_kicad"
         (path "/729eee83-acb9-4794-a583-aef43df0c6ef"
           (reference "C3") (unit 1)
@@
     (pin "6")
     (instances
-      (project "skateboard_main_controller"
+      (project "skateboard_main_controller_kicad"
         (path "/729eee83-acb9-4794-a583-aef43df0c6ef"
           (reference "J2") (unit 1)
@@
     (pin "1")
     (instances
-      (project "skateboard_main_controller"
+      (project "skateboard_main_controller_kicad"
         (path "/729eee83-acb9-4794-a583-aef43df0c6ef"
           (reference "TP2") (unit 1)
@@
     (pin "1")
     (instances
-      (project "skateboard_main_controller"
+      (project "skateboard_main_controller_kicad"
         (path "/729eee83-acb9-4794-a583-aef43df0c6ef"
           (reference "#PWR01") (unit 1)
@@
     (pin "1")
     (instances
-      (project "skateboard_main_controller"
+      (project "skateboard_main_controller_kicad"
         (path "/729eee83-acb9-4794-a583-aef43df0c6ef"
           (reference "J4") (unit 1)
@@
     (pin "1")
     (instances
-      (project "skateboard_main_controller"
+      (project "skateboard_main_controller_kicad"
         (path "/729eee83-acb9-4794-a583-aef43df0c6ef"
           (reference "#PWR08") (unit 1)
@@
     (pin "2")
     (instances
-      (project "skateboard_main_controller"
+      (project "skateboard_main_controller_kicad"
         (path "/729eee83-acb9-4794-a583-aef43df0c6ef"
           (reference "C1") (unit 1)
@@
     (pin "1")
     (instances
-      (project "skateboard_main_controller"
+      (project "skateboard_main_controller_kicad"
         (path "/729eee83-acb9-4794-a583-aef43df0c6ef"
           (reference "#PWR012") (unit 1)
@@
     (pin "1")
     (instances
-      (project "skateboard_main_controller"
+      (project "skateboard_main_controller_kicad"
         (path "/729eee83-acb9-4794-a583-aef43df0c6ef"
           (reference "#PWR02") (unit 1)
@@
     (pin "1")
     (instances
-      (project "skateboard_main_controller"
+      (project "skateboard_main_controller_kicad"
         (path "/729eee83-acb9-4794-a583-aef43df0c6ef"
           (reference "#PWR09") (unit 1)
@@
     (pin "1")
     (instances
-      (project "skateboard_main_controller"
+      (project "skateboard_main_controller_kicad"
         (path "/729eee83-acb9-4794-a583-aef43df0c6ef"
           (reference "#PWR07") (unit 1)
@@
     (pin "9")
     (instances
-      (project "skateboard_main_controller"
+      (project "skateboard_main_controller_kicad"
         (path "/729eee83-acb9-4794-a583-aef43df0c6ef"
           (reference "MT1") (unit 1)
@@
     (pin "1")
     (instances
-      (project "skateboard_main_controller"
+      (project "skateboard_main_controller_kicad"
         (path "/729eee83-acb9-4794-a583-aef43df0c6ef"
           (reference "#PWR013") (unit 1)
@@
     (pin "1")
     (instances
-      (project "skateboard_main_controller"
+      (project "skateboard_main_controller_kicad"
         (path "/729eee83-acb9-4794-a583-aef43df0c6ef"
           (reference "#PWR06") (unit 1)
@@
     (pin "2")
     (instances
-      (project "skateboard_main_controller"
+      (project "skateboard_main_controller_kicad"
         (path "/729eee83-acb9-4794-a583-aef43df0c6ef"
           (reference "C2") (unit 1)
@@
     (pin "1")
     (instances
-      (project "skateboard_main_controller"
+      (project "skateboard_main_controller_kicad"
         (path "/729eee83-acb9-4794-a583-aef43df0c6ef"
           (reference "#PWR04") (unit 1)
@@
     (pin "2")
     (instances
-      (project "skateboard_main_controller"
+      (project "skateboard_main_controller_kicad"
         (path "/729eee83-acb9-4794-a583-aef43df0c6ef"
           (reference "C8") (unit 1)

Commit message: PCB initial commit
Parts:
- C1, C2, C3, C4, C5, C6, C7, C8: footprint (none) -> Capacitor_SMD:C_0805_2012Metric
- J1: footprint (none) -> Connector_PinHeader_2.54mm:PinHeader_1x02_P2.54mm_Vertical
- J2: footprint (none) -> Connector_PinHeader_2.54mm:PinHeader_1x06_P2.54mm_Vertical
- J3, J4: footprint (none) -> Connector_PinHeader_2.54mm:PinHeader_1x01_P2.54mm_Vertical
- MT1: footprint ICM-42670-P:XDCR_ICM-42670-P -> STM32:XDCR_ICM-42670-P
- TP1, TP2, TP3, TP4: footprint (none) -> TestPoint:TestPoint_Keystone_5010-5014_Multipurpose
- U1: footprint STM32F103C8T6TR:QFP50P900X900X160-48N -> STM32:QFP50P900X900X160-48N
