File: skateboard_main_controller_kicad/skateboard_main_controller_kicad.kicad_pcb (KiCad board)
At the start: 2 copper layers, 99.9 x 99.9 mm, 22 parts, among them J1 Conn_01x02_Socket, J2 Conn_01x06_Socket, J3 Conn_01x01_Socket, J4 Conn_01x01_Socket, U1 STM32F103C8T6TR

Commit message: PCB_V2
Parts:
- removed J3: Conn_01x01_Socket, Connector_PinHeader_2.54mm:PinHeader_1x01_P2.54mm_Vertical
- added C10: 100n, Capacitor_SMD:C_0805_2012Metric, B.Cu at (189.5, 63.1)
- added C11: 1u, Capacitor_SMD:C_0805_2012Metric, F.Cu at (223.5, 55.9)
- added C12: 1u, Capacitor_SMD:C_0805_2012Metric, F.Cu at (215.3, 59.7)
- added C9: 100n, Capacitor_SMD:C_0805_2012Metric, B.Cu at (184.5, 61.5)
- added GND1: TestPoint, TestPoint:TestPoint_Keystone_5010-5014_Multipurpose, F.Cu at (145.8, 83.5)
- added GND2: TestPoint, TestPoint:TestPoint_Keystone_5010-5014_Multipurpose, F.Cu at (145.8, 91.3)
- added J5: Conn_01x02_Pin, Connector_PinHeader_2.54mm:PinHeader_1x02_P2.54mm_Vertical, F.Cu at (188.6, 37.6)
- added J6: Conn_02x10_Odd_Even, Connector_PinHeader_2.54mm:PinHeader_2x10_P2.54mm_Vertical, F.Cu at (194.1, 37.6)
- added J7: Conn_01x02_Pin, Connector_PinHeader_2.54mm:PinHeader_1x02_P2.54mm_Vertical, F.Cu at (224.8, 43.2)
- added J8: Conn_01x02_Pin, Connector_PinHeader_2.54mm:PinHeader_1x02_P2.54mm_Vertical, F.Cu at (222.2, 51.3)
- added R1: 10k, Resistor_SMD:R_0805_2012Metric, F.Cu at (187.3, 55.4)
- added R2: 10k, Resistor_SMD:R_0805_2012Metric, F.Cu at (166.6, 77.7)
- added U2: AP2112K-3.3, Package_TO_SOT_SMD:SOT-23-5, F.Cu at (219.6, 58.4)
- C1, C2, C3, C4, C5, C6, C7, C8: moved to F.Cu
- moved MOSI1 51.7 mm to (153.9, 91.3)
- moved SCLK1 43.4 mm to (153.9, 83.5)
- moved SPI_CS1 39.3 mm to (153.9, 75.7)
- moved C4 20.8 mm to (183.8, 57.9), turned to 180 degrees
- moved J1 15.1 mm to (204.7, 101.1)
- moved MISO1 13.7 mm to (153.9, 99.1)
- moved C7 10.0 mm to (189.0, 79.3), turned to 90 degrees
- moved C6 9.77 mm to (186.9, 79.3), turned to 90 degrees
- moved C3 9.17 mm to (196.1, 59.9), turned to 0 degrees
- moved C5 7.75 mm to (179.1, 58.7), turned to 90 degrees
- moved C2 3.38 mm to (194.1, 67.6), turned to 0 degrees
- moved C8 3.18 mm to (190.5, 85.1), turned to 0 degrees
- moved C1 1.40 mm to (181.8, 64.0), turned to 180 degrees
- renumbered TP1 to MISO1, TP4 to MOSI1, TP2 to SCLK1, TP3 to SPI_CS1
Connections:
- J2 pad 2: CTS -> Net-(J2-Pin_2)
- J2 pad 3: VCC -> unconnected-(J2-Pin_3-Pad3)
- J2 pad 6: DTR -> unconnected-(J2-Pin_6-Pad6)
- MT1 pad 4: unconnected-(MT1-INT1/INT-Pad4) -> INT1
- U1 pad 1: unconnected-(U1-VBAT-Pad1) -> Net-(U1-VBAT)
- U1 pad 13: unconnected-(U1-PA3-Pad13) -> INT1
- U1 pad 32: CTS -> unconnected-(U1-PA11-Pad32)
- U1 pad 34: unconnected-(U1-PA13-Pad34) -> SWDIO
- U1 pad 37: unconnected-(U1-PA14-Pad37) -> SWCLK
- U1 pad 39: unconnected-(U1-PB3-Pad39) -> SWO
- U1 pad 44: VCC -> Net-(J5-Pin_1)
- U1 pad 7: DTR -> NRST
Routing:
- net NRST: track 0.00 -> 54.4 mm, vias 0 -> 3
- net VCC: track 75.3 -> 21.6 mm, vias 6 -> 1
- net DTR: track 46.7 -> 0.00 mm
- net SWO: track 0.00 -> 38.5 mm, vias 0 -> 1
- net CTS: track 36.7 -> 0.00 mm
- net SWDIO: track 0.00 -> 31.0 mm, vias 0 -> 1
- net SWCLK: track 0.00 -> 28.0 mm, vias 0 -> 2
- net MISO: track 86.4 -> 61.8 mm
- net INT1: track 0.00 -> 23.7 mm, vias 0 -> 2
- net Net-(J5-Pin_1): track 0.00 -> 23.1 mm, vias 0 -> 1
- net GND: track 24.2 -> 45.3 mm, vias 4 -> 12
- net Net-(J2-Pin_2): track 0.00 -> 18.6 mm
- net ADC12_IN8: track 23.2 -> 38.3 mm
- net Net-(J8-Pin_2): track 0.00 -> 13.0 mm
- net unconnected-(J7-Pin_1-Pad1): track 0.00 -> 10.4 mm
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Other:
- board text added: "ADC_IN"
- board text added: "BOOT0"
- board text added: "PWM"
- board text added: "USB | Battery"

Commit message: Screw_Termal
Parts:
- added J3: 39543-0602, STM32:SHDR2W100P0X500_1X2_1000X760X1040P, F.Cu at (235.0, 43.4)
Connections:
- J7 pad 1: unconnected-(J7-Pin_1-Pad1) -> Net-(J7-Pin_1)
Routing:
- net unconnected-(J7-Pin_1-Pad1): track 10.4 -> 0.00 mm
- net Net-(J7-Pin_1): track 0.00 -> 10.4 mm
Other:
- board text added: "+"
- board text added: "-"

Commit message: v3
Parts:
- added J9: Conn_01x02_Socket, Connector_PinHeader_2.54mm:PinHeader_1x02_P2.54mm_Vertical, F.Cu at (222.4, 101.1)
Connections:
- U1 pad 19: unconnected-(U1-PB1-Pad19) -> ADC12_IN9
Routing:
- net ADC12_IN9: track 0.00 -> 46.7 mm
Other:
- board text added: "ADC_IN2"
