File: skateboard_main_controller_kicad/.history/skateboard_main_controller_kicad.kicad_pcb (KiCad board)
At the start: 2 copper layers, 18 parts, among them J1 Conn_01x02_Socket, J2 Conn_01x06_Socket, J3 Conn_01x01_Socket, J4 Conn_01x01_Socket, U1 STM32F103C8T6TR

Commit message: hello
Parts:
- C1, C2, C3, C4, C5, C6, C7, C8: moved to B.Cu
- moved J2 120.6 mm to (228.7, 57.0)
- moved C4 105.8 mm to (203.2, 65.4), turned to -90 degrees
- moved C2 97.5 mm to (196.7, 65.4), turned to -90 degrees
- moved C7 96.0 mm to (197.1, 85.2), turned to -90 degrees
- moved J3 94.6 mm to (186.3, 37.6)
- moved TP4 91.8 mm to (203.2, 106.9), turned to 90 degrees
- moved C3 91.5 mm to (188.7, 65.4), turned to -90 degrees
- moved C8 88.2 mm to (187.3, 85.1), turned to -90 degrees
- moved U1 84.6 mm to (189.0, 62.7)
- moved C5 83.0 mm to (175.1, 65.4), turned to -90 degrees
- moved C1 82.6 mm to (181.7, 65.4), turned to -90 degrees
- moved TP2 78.5 mm to (190.5, 106.9), turned to 90 degrees
- moved C6 78.2 mm to (179.1, 85.1), turned to -90 degrees
- moved J1 71.4 mm to (203.8, 86.0), turned to 180 degrees
- moved TP3 66.0 mm to (177.8, 106.9), turned to 90 degrees
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Routing:
- net MISO: track 0.00 -> 80.2 mm, vias 0 -> 2
- net MOSI: track 0.00 -> 54.2 mm
- net VCC: track 0.00 -> 49.5 mm, vias 0 -> 2
- net DTR: track 0.00 -> 46.7 mm
- net SPI_CS: track 0.00 -> 46.6 mm
- net SCK: track 0.00 -> 45.2 mm, vias 0 -> 2
- net RX_laptop: track 0.00 -> 37.3 mm
- net CTS: track 0.00 -> 36.7 mm
- net TX_laptop: track 0.00 -> 36.6 mm
- net Net-(J4-Pin_1): track 0.00 -> 28.6 mm
- net ADC12_IN8: track 0.00 -> 23.2 mm
- net GND: track 0.00 -> 4.90 mm, vias 0 -> 3
Other:
- board outline added: 99.9 x 99.9 mm

Commit message: JLKDJF
Parts:
- added REF**: MountingHole_3.2mm_M3, MountingHole:MountingHole_3.2mm_M3, F.Cu at (230.5, 114.2)
- added REF**: MountingHole_3.2mm_M3, MountingHole:MountingHole_3.2mm_M3, F.Cu at (230.5, 34.3)
- added REF**: MountingHole_3.2mm_M3, MountingHole:MountingHole_3.2mm_M3, F.Cu at (150.6, 34.3)
- added REF**: MountingHole_3.2mm_M3, MountingHole:MountingHole_3.2mm_M3, F.Cu at (150.6, 114.2)
Routing:
- net VCC: track 49.5 -> 75.3 mm, vias 2 -> 6
- net GND: track 4.90 -> 24.2 mm, vias 3 -> 4
- net MISO: track 80.2 -> 86.4 mm
- added copper zone on B.Cu, net GND
- added copper zone on F.Cu, net VCC
