File: skateboard_main_controller_kicad/.history/skateboard_main_controller_kicad.kicad_sch (KiCad schematic)
At the start: 18 parts, among them J1 Conn_01x02_Socket, J2 Conn_01x06_Socket, J3 Conn_01x01_Socket, J4 Conn_01x01_Socket, U1 STM32F103C8T6TR

Commit message: PCB_V2
Parts:
- removed J3: Conn_01x01_Socket, Connector_PinHeader_2.54mm:PinHeader_1x01_P2.54mm_Vertical, symbol Connector:Conn_01x01_Socket
- added C10, C9: 100n, Capacitor_SMD:C_0805_2012Metric, symbol Device:C
- added C11, C12: 1u, Capacitor_SMD:C_0805_2012Metric, symbol Device:C
- added GND1, GND2: TestPoint, TestPoint:TestPoint_Keystone_5010-5014_Multipurpose, symbol Connector:TestPoint
- added J5: Conn_01x02_Pin, symbol Connector:Conn_01x02_Pin
- added J6: Conn_02x10_Odd_Even, Connector_PinHeader_2.54mm:PinHeader_2x10_P2.54mm_Vertical, symbol Connector_Generic:Conn_02x10_Odd_Even
- added J7, J8: Conn_01x02_Pin, Connector_PinHeader_2.54mm:PinHeader_1x02_P2.54mm_Vertical, symbol Connector:Conn_01x02_Pin
- added R1, R2: 10k, Resistor_SMD:R_0805_2012Metric, symbol Device:R_US
- added U2: AP2112K-3.3, Package_TO_SOT_SMD:SOT-23-5, symbol Regulator_Linear:AP2112K-3.3
- renumbered TP1 to MISO1, TP4 to MOSI1, TP2 to SCLK1, TP3 to SPI_CS1
Connections:
- net +3.3V: now also C10.2, J5.2 (Pin_2), J6.1 (Pin_1), J6.2 (Pin_2), J7.2 (Pin_2), J8.1 (Pin_1), R2.1; no longer J2.3 (Pin_3), U1.44 (BOOT0)
- net GND: now also C11.2, C12.2, C9.1, GND1.1, GND2.1, J6.10 (Pin_10), J6.12 (Pin_12), J6.14 (Pin_14), J6.16 (Pin_16), J6.18 (Pin_18), J6.20 (Pin_20), J6.3 (Pin_3), J6.4 (Pin_4), J6.5 (Pin_5), J6.6 (Pin_6), J6.8 (Pin_8), R1.1, U2.2 (GND)
- net SPI_CS: now also R2.2
- net at U1.1 (VBAT): now also C10.1
- net INT1: now reaches U1.13 (PA3)
- net INT1: now also MT1.4 (INT1/INT)
- net SWDIO: now reaches U1.34 (PA13)
- net SWDIO: now also J6.7 (Pin_7)
- net SWCLK: now reaches U1.37 (PA14)
- net SWCLK: now also J6.9 (Pin_9)
- net SWO: now reaches U1.39 (PB3)
- net SWO: now also J6.13 (Pin_13)
- net CTS: no longer names the net of J2.2 (Pin_2)
- net CTS: now also C11.1, U2.1 (VIN), U2.3 (EN); no longer U1.32 (PA11)
- net DTR: no longer names the net of J2.6 (Pin_6)
- net DTR: no longer U1.7 (NRST)
- new net: C12.1, J8.2 (Pin_2), U2.5 (VOUT)
- new net: J5.1 (Pin_1), R1.2, U1.44 (BOOT0)
- new net NRST: C9.2, J6.15 (Pin_15), U1.7 (NRST)
- no-connect marks 4 -> 34
Other:
- moved on the sheet: J2

Commit message: Screw_Termal
Parts:
- added J3: 39543-0602, SHDR2W100P0X500_1X2_1000X760X1040P, symbol Screw_Terminal:39543-0602
Connections:
- net GND: now also J3.2
- net at J7.1 (Pin_1): now also J3.1
Changed lines of the file:
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@@
+	)
+	(symbol
+		(lib_id "Screw_Terminal:39543-0602")
+		(at 258.445 124.46 0)
+		(unit 1)
+		(body_style 1)
+		(exclude_from_sim no)
+		(in_bom yes)
+		(on_board yes)
+		(in_pos_files yes)
+		(dnp no)
+		(fields_autoplaced yes)
+		(property "Reference" "J3"
+			(at 275.59 124.4599 0)
+			(show_name no)
+			(do_not_autoplace no)
+			(effects
+				(font
+					(size 1.27 1.27)
+				)
+				(justify left)
+			)
+		)
+		(property "Value" "39543-0602"
+			(at 275.59 126.9999 0)
+			(show_name no)
+			(do_not_autoplace no)
+			(effects
+				(font
+					(size 1.27 1.27)
+				)
+				(justify left)
+			)
+		)
+		(property "Footprint" "SHDR2W100P0X500_1X2_1000X760X1040P"
+			(at 274.955 219.38 0)
+			(hide yes)
+			(show_name no)
+			(do_not_autoplace no)
+			(effects
+				(font
+					(size 1.27 1.27)
+				)
+				(justify left top)
+			)
+		)
+		(property "Datasheet" "https://componentsearchengine.com/Datasheets/1/39543-0602.pdf"
+			(at 274.955 319.38 0)
+			(hide yes)
+			(show_name no)
+			(do_not_autoplace no)
+			(effects
+				(font
+					(size 1.27 1.27)
+				)
+				(justify left top)
+			)
+		)
+		(property "Description" "Fixed Terminal Blocks 5.0MM EUROBLOCK PC VERT LP BLK 2CKT"
+			(at 258.445 124.46 0)
+			(hide yes)
+			(show_name no)
+			(do_not_autoplace no)
+			(effects
+				(font
+					(size 1.27 1.27)
+				)
+			)
+		)
+		(property "Height" "10.4"
+			(at 274.955 519.38 0)
+			(hide yes)
+			(show_name no)
+			(do_not_autoplace no)
+			(effects
+				(font
+					(size 1.27 1.27)
+				)
+				(justify left top)
+			)
+		)
+		(property "Mouser Part Number" "538-39543-0602"
+			(at 274.955 619.38 0)
+			(hide yes)
+			(show_name no)
+			(do_not_autoplace no)
+			(effects
+				(font
+					(size 1.27 1.27)
+				)
+				(justify left top)
+			)
+		)
+		(property "Mouser Price/Stock" "https://www.mouser.co.uk/ProductDetail/Molex/39543-0602?qs=4dAX1jW9NQoaQAX2Pqen2w%3D%3D"
+			(at 274.955 719.38 0)
+			(hide yes)
+			(show_name no)
+			(do_not_autoplace no)
+			(effects
+				(font
+					(size 1.27 1.27)
+				)
+				(justify left top)
+			)
+		)
+		(property "Manufacturer_Name" "Molex"
+			(at 274.955 819.38 0)
+			(hide yes)
+			(show_name no)
+			(do_not_autoplace no)
+			(effects
+				(font
+					(size 1.27 1.27)
+				)
+				(justify left top)
+			)
+		)
+		(property "Manufacturer_Part_Number" "39543-0602"
+			(at 274.955 919.38 0)
+			(hide yes)
+			(show_name no)
+			(do_not_autoplace no)
+			(effects
+				(font
+					(size 1.27 1.27)
+				)
+				(justify left top)
+			)
+		)
+		(pin "1"
+		)
+		(pin "2"
+		)
+		(instances
+			(project "skateboard_main_controller_kicad"
+				(path "/729eee83-acb9-4794-a583-aef43df0c6ef"
+					(reference "J3")
+					(unit 1)
+				)
+			)
+		)
 	)
 	(symbol

Commit message: v3
Parts:
- added J9: Conn_01x02_Socket, Connector_PinHeader_2.54mm:PinHeader_1x02_P2.54mm_Vertical, symbol Connector:Conn_01x02_Socket
Connections:
- net GND: now also J9.1 (Pin_1)
- net ADC12_IN9: now reaches U1.19 (PB1)
- net ADC12_IN9: now also J9.2 (Pin_2)
- no-connect marks 34 -> 33
Other:
- note added: "ADC In Socket"
Changed lines of the file:
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@@
 		)
 	)
+	(text "ADC In Socket\n"
+		(exclude_from_sim no)
+		(at 285.75 273.558 0)
+		(effects
+			(font
+				(size 1.27 1.27)
+			)
+		)
+	)
 	(junction
 		(at 298.45 165.735)
@@
 	)
 	(no_connect
-		(at 278.765 187.325)
-	)
-	(no_connect
 		(at 278.765 210.185)
 	)
@@
 		)
 	)
+	(global_label "ADC12_IN9"
+		(shape input)
+		(at 274.955 278.765 180)
+		(fields_autoplaced yes)
+		(effects
+			(font
+				(size 1.27 1.27)
+			)
+			(justify right)
+		)
+		(property "Intersheetrefs" "${INTERSHEET_REFS}"
+			(at 261.8098 278.765 0)
+			(hide yes)
+			(show_name no)
+			(do_not_autoplace no)
+			(effects
+				(font
+					(size 1.27 1.27)
+				)
+				(justify right)
+			)
+		)
+	)
 	(global_label "INT1"
 		(shape input)
@@
 		)
 	)
+	(global_label "ADC12_IN9"
+		(shape input)
+		(at 278.765 187.325 0)
+		(fields_autoplaced yes)
+		(effects
+			(font
+				(size 1.27 1.27)
+			)
+			(justify left)
+		)
+		(property "Intersheetrefs" "${INTERSHEET_REFS}"
+			(at 291.9102 187.325 0)
+			(hide yes)
+			(show_name no)
+			(do_not_autoplace no)
+			(effects
+				(font
+					(size 1.27 1.27)
+				)
+				(justify left)
+			)
+		)
+	)
 	(global_label "RX_laptop"
 		(shape input)
@@
 	)
 	(symbol
+		(lib_name "GND_8")
+		(lib_id "power:GND")
+		(at 274.955 276.225 180)
+		(unit 1)
+		(body_style 1)
+		(exclude_from_sim no)
+		(in_bom yes)
+		(on_board yes)
+		(in_pos_files yes)
+		(dnp no)
+		(fields_autoplaced yes)
+		(property "Reference" "#PWR023"
+			(at 274.955 269.875 0)
+			(hide yes)
+			(show_name no)
+			(do_not_autoplace no)
+			(effects
+				(font
+					(size 1.27 1.27)
+				)
+			)
+		)
+		(property "Value" "GND"
+			(at 274.955 271.78 0)
+			(show_name no)
+			(do_not_autoplace no)
+			(effects
+				(font
+					(size 1.27 1.27)
+				)
+			)
+		)
+		(property "Footprint" ""
+			(at 274.955 276.225 0)
+			(hide yes)
+			(show_name no)
+			(do_not_autoplace no)
+			(effects
+				(font
+					(size 1.27 1.27)
+				)
+			)
+		)
+		(property "Datasheet" ""
+			(at 274.955 276.225 0)
+			(hide yes)
+			(show_name no)
+			(do_not_autoplace no)
+			(effects
+				(font
+					(size 1.27 1.27)
+				)
+			)
+		)
+		(property "Description" "Power symbol creates a global label with name \"GND\" , ground"
+			(at 274.955 276.225 0)
+			(hide yes)
+			(show_name no)
+			(do_not_autoplace no)
+			(effects
+				(font
+					(size 1.27 1.27)
+				)
+			)
+		)
+		(pin "1"
+		)
+		(instances
+			(project "skateboard_main_controller_kicad"
+				(path "/729eee83-acb9-4794-a583-aef43df0c6ef"
+					(reference "#PWR023")
+					(unit 1)
+				)
+			)
+		)
+	)
+	(symbol
 		(lib_name "+3.3V_2")
 		(lib_id "power:+3.3V")
@@
 					(unit 1)
 				)
+			)
+		)
+	)
+	(symbol
+		(lib_id "Connector:Conn_01x02_Socket")
+		(at 280.035 276.225 0)
+		(unit 1)
+		(body_style 1)
+		(exclude_from_sim no)
+		(in_bom yes)
+		(on_board yes)
+		(in_pos_files yes)
+		(dnp no)
+		(property "Reference" "J9"
+			(at 276.86 283.845 0)
+			(show_name no)
+			(do_not_autoplace no)
+			(effects
+				(font
+					(size 1.27 1.27)
+				)
+				(justify left)
+			)
+		)
+		(property "Value" "Conn_01x02_Socket"
+			(at 268.605 281.94 0)
+			(show_name no)
+			(do_not_autoplace no)
+			(effects
+				(font
+					(size 1.27 1.27)
+				)
+				(justify left)
+			)
+		)
+		(property "Footprint" "Connector_PinHeader_2.54mm:PinHeader_1x02_P2.54mm_Vertical"
+			(at 280.035 276.225 0)
+			(hide yes)
+			(show_name no)
+			(do_not_autoplace no)
+			(effects
+				(font
+					(size 1.27 1.27)
+				)
+			)
+		)
+		(property "Datasheet" ""
+			(at 280.035 276.225 0)
+			(hide yes)
+			(show_name no)
+			(do_not_autoplace no)
+			(effects
+				(font
+					(size 1.27 1.27)
+				)
+			)
+		)
+		(property "Description" ""
+			(at 280.035 276.225 0)
+			(show_name no)
+			(do_not_autoplace no)
+			(effects
+				(font
+					(size 1.27 1.27)
+				)
+			)
+		)
+		(pin "1"
+		)
+		(pin "2"
+		)
+		(instances
+			(project "skateboard_main_controller_kicad"
+				(path "/729eee83-acb9-4794-a583-aef43df0c6ef"
+					(reference "J9")
+					(unit 1)
+				)
